File: CPU_ESP/V0.4/CPU/I2C.kicad_sch (KiCad schematic)
At the start: 32 parts, among them U201 LM75A, U202 PCA9306, U203 PCF8563T, U204 TCA9544A, U205 MCP23017_SS, U207 AT24CS01-SSHM, Y201 32.278kHz

Commit message: Update I2C Adresse
Parts:
- U207: value AT24CS01-SSHM -> 24FC-1025
Other:
- note added: "I2C ADRESSE : 0X20"
- note added: "I2C ADRESSE : 0X48"
- note added: "I2C ADRESSE : 0X50"
- note added: "I2C ADRESSE : 0X51"
- note added: "I2C ADRESSE : 0X70"
Changed lines of the file:
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@@
 		(comment 1 "I2C")
 	)
+	(text "I2C ADRESSE : 0X48"
+		(exclude_from_sim no)
+		(at 37.338 83.058 0)
+		(effects
+			(font
+				(size 1.27 1.27)
+			)
+		)
+	)
+	(text "I2C ADRESSE : 0X20"
+		(exclude_from_sim no)
+		(at 177.8 97.79 0)
+		(effects
+			(font
+				(size 1.27 1.27)
+			)
+		)
+	)
+	(text "I2C ADRESSE : 0X70"
+		(exclude_from_sim no)
+		(at 188.722 18.034 0)
+		(effects
+			(font
+				(size 1.27 1.27)
+			)
+		)
+	)
+	(text "I2C ADRESSE : 0X51"
+		(exclude_from_sim no)
+		(at 55.626 29.464 0)
+		(effects
+			(font
+				(size 1.27 1.27)
+			)
+		)
+	)
 	(text "REAL TIME CLOCK"
 		(exclude_from_sim no)
@@
 		)
 	)
+	(text "I2C ADRESSE : 0X50"
+		(exclude_from_sim no)
+		(at 256.286 72.898 0)
+		(effects
+			(font
+				(size 1.27 1.27)
+			)
+		)
+	)
 	(junction
 		(at 27.94 160.02)
@@
 			)
 		)
-		(property "Value" "AT24CS01-SSHM"
+		(property "Value" "24FC-1025"
 			(at 258.6833 82.55 0)
 			(effects
