File: CPU_ESP/V0.4/CPU/sevensegments.kicad_sch (KiCad schematic)
At the start: 7 parts, among them Q601 BSR19, Q602 BSR19, U601 SAA1064T

Commit message: Update I2C Adresse
Other:
- note added: "I2C ADRESSE : 0X38"
Changed lines of the file:
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@@
 		(comment 1 "SEVEN SEGMENTS")
+	)
+	(text "I2C ADRESSE : 0X38"
+		(exclude_from_sim no)
+		(at 135.636 59.69 0)
+		(effects
+			(font
+				(size 1.27 1.27)
+			)
+		)
 	)
 	(junction
